File: KiCad/steg_7.kicad_sch (KiCad schematic)
At the start: 14 parts, among them U1 W65C02S, U2 LCD-016N002L, U3 W65C22, U4 74HC00

Commit message: Kicad projekt ligger här nu, med alla steg
Parts:
- added C7, C8: 100nF, symbol Device:C_Small
- A1: value Arduino_Mega2560_R3_Shield -> Mega2560
- U2: value LCD-016N002L -> LCD
Connections:
- net +5V: now also C7.1, C8.1
- net Earth: now also U2.5 (R/~{W}), C7.2, C8.2
- net at U3.3 (PA1): no longer U2.5 (R/~{W})
